File: CH32V203-DevBoard.kicad_sch (KiCad schematic)
At the start: 41 parts, among them J1 USB_C_Receptacle_USB2.0_16P, J2 USB_C_Receptacle_USB2.0_16P, Q1 AO3401A, Q2 AO3401A, SW1 SW_Push, SW2 SW_Push, U1 CH32V203C8T6, U2 RT9080-33GJ5

Commit message: fix rotation offset and readme
Parts:
- D2: JLCPCB Rotation Offset -180 -> 0
- Q1, Q2: JLCPCB Rotation Offset 180 -> 0
- U1: JLCPCB Rotation Offset -90 -> 0
Changed lines of the file:
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@@
 			)
 		)
-		(property "JLCPCB Rotation Offset" "180"
+		(property "JLCPCB Rotation Offset" "0"
 			(at 215.9 36.83 90)
 			(effects
@@
 			)
 		)
-		(property "JLCPCB Rotation Offset" "180"
+		(property "JLCPCB Rotation Offset" "0"
 			(at 205.74 36.83 90)
 			(effects
@@
 			)
 		)
-		(property "JLCPCB Rotation Offset" "-180"
+		(property "JLCPCB Rotation Offset" "0"
 			(at 256.54 137.16 0)
 			(effects
@@
 			)
 		)
-		(property "JLCPCB Rotation Offset" "-90"
+		(property "JLCPCB Rotation Offset" "0"
 			(at 46.99 139.7 0)
 			(effects
